File: Wiring_Diagram/kiCAD_files/ChickenDoor-kiCAD.sch (KiCad schematic (older format))
At the start: 10 parts

Commit message: Add files via upload
Parts:
- removed SW_Toggle-auto-or-manual: SW_Push_DPDT, symbol Switch:SW_Push_DPDT
- added SW_Toggle-auto-or-manual?: SW_Push_DPDT, symbol Switch:SW_Push_DPDT
- A?: symbol MCU_Module:Arduino_UNO_R3 -> ChickenDoor-kiCAD-rescue:Arduino_UNO_R3-MCU_Module
Connections:
- net at 12VDC.1 (+), EMERGENCYSTOP.1 (A): now also K?.3 (NO1)
- net at K?.4 (NC2): now also SW_RockerSW_manual_moto_ctl.4
- net at EMERGENCYSTOP.2 (B): now also SW_RockerSW_manual_moto_ctl.6
- new net: M_LInear_Actuator.1 (+), SW_Toggle-auto-or-manual?.2 (B)
- new net: M_LInear_Actuator.2 (-), SW_Toggle-auto-or-manual?.5 (B)
- new net: K?.1 (COM1), SW_Toggle-auto-or-manual?.6 (C)
- new net: K?.2 (COM0), SW_Toggle-auto-or-manual?.3 (C)
- new net: SW_RockerSW_manual_moto_ctl.2, SW_Toggle-auto-or-manual?.1 (A)
- new net: SW_RockerSW_manual_moto_ctl.5, SW_Toggle-auto-or-manual?.4 (A)
Other:
- moved on the sheet: M_LInear_Actuator
Changed lines of the file:
@@
 EESchema Schematic File Version 4
+LIBS:ChickenDoor-kiCAD-cache
 EELAYER 30 0
 EELAYER END
@@
 $EndDescr
 $Comp
-L MCU_Module:Arduino_UNO_R3 A?
+L ChickenDoor-kiCAD-rescue:Arduino_UNO_R3-MCU_Module A?
 U 1 1 5DE0B9A7
 P 7750 3050
@@
 L Motor:Motor_DC M_LInear_Actuator
 U 1 1 5DE0D523
-P 2800 4350
-F 0 "M_LInear_Actuator" H 2958 4346 50  0000 L CNN
-F 1 "Motor_DC" H 2958 4255 50  0000 L CNN
-F 2 "" H 2800 4260 50  0001 C CNN
-F 3 "~" H 2800 4260 50  0001 C CNN
-	1    2800 4350
-	1    0    0    -1
+P 2850 5150
+F 0 "M_LInear_Actuator" H 3008 5146 50  0000 L CNN
+F 1 "Motor_DC" H 3008 5055 50  0000 L CNN
+F 2 "" H 2850 5060 50  0001 C CNN
+F 3 "~" H 2850 5060 50  0001 C CNN
+	1    2850 5150
+	0    -1   -1   0
 $EndComp
 $Comp
@@
 $EndComp
 Wire Wire Line
-	2800 4650 4250 4650
-Wire Wire Line
-	4250 3850 4150 3850
-Wire Wire Line
 	4850 4350 5000 4350
 Wire Wire Line
-	5000 4350 5000 4700
-Wire Wire Line
 	5000 4750 4850 4750
-Wire Wire Line
-	5000 4700 5650 4700
-Connection ~ 5000 4700
-Wire Wire Line
-	5000 4700 5000 4750
-Wire Wire Line
-	5650 4700 5650 2900
-Wire Wire Line
-	5650 2900 4150 2900
-Wire Wire Line
-	4150 2900 4150 3850
 Wire Wire Line
 	4850 3450 6200 3450
@@
 Connection ~ 9850 3400
 Wire Wire Line
-	4250 4250 3200 4250
-Wire Wire Line
 	4850 4150 4900 4150
 Wire Wire Line
@@
 Wire Wire Line
 	3800 2350 3700 2350
-Connection ~ 4150 3850
 Entry Wire Line
 	5650 2750 5750 2850
@@
 Entry Wire Line
 	4050 2750 4150 2650
-Wire Wire Line
-	2200 3800 2200 4650
-Wire Wire Line
-	2200 4650 2800 4650
-Connection ~ 2800 4650
-Wire Wire Line
-	2800 4150 3200 4150
-Wire Wire Line
-	3200 4150 3200 4250
-$Comp
-L Switch:SW_Push_DPDT SW_Toggle-auto-or-manual
-U 1 1 5DF7A4F3
-P 3900 1500
-F 0 "SW_Toggle-auto-or-manual" V 3946 1112 50  0000 R CNN
-F 1 "SW_Push_DPDT" V 3855 1112 50  0000 R CNN
-F 2 "" H 3900 1700 50  0001 C CNN
-F 3 "~" H 3900 1700 50  0001 C CNN
-	1    3900 1500
-	0    -1   -1   0
-$EndComp
-Wire Wire Line
-	4100 2350 4100 1700
-Wire Wire Line
-	4000 1300 4000 1200
-Wire Wire Line
-	4000 1200 4300 1200
-Wire Wire Line
-	4300 1200 4300 2650
-Wire Wire Line
-	4300 2650 4150 2650
-Wire Wire Line
-	3300 2350 3300 1700
-Wire Wire Line
-	4200 1300 4200 1100
-Wire Wire Line
-	4200 1100 2700 1100
-Wire Wire Line
-	2700 1100 2700 3400
-Wire Wire Line
-	3800 1300 3800 1200
-Wire Wire Line
-	3800 1200 2500 1200
-Wire Wire Line
-	2500 1200 2500 3400
-Wire Wire Line
-	3300 1700 3700 1700
-Wire Wire Line
-	3600 1300 3100 1300
-Wire Wire Line
-	3100 1300 3100 3850
-Wire Wire Line
-	3100 3850 4150 3850
-Wire Wire Line
-	2800 4150 2600 4150
-Wire Wire Line
-	2600 4150 2600 3800
-Connection ~ 2800 4150
 $Comp
 L sensor_optical_ir_breakbeam_sensor:Sensor_Optical_IR_breakbeam_Sensor U?
@@
 Wire Wire Line
 	6000 3150 7250 3150
-Wire Bus Line
-	4050 2750 5800 2750
 $Comp
 L sw_dpdt_msm_center-off:SW_DPDT_MSM_Center-OFF SW_RockerSW_manual_moto_ctl
@@
 	0    1    1    0
 $EndComp
+$Comp
+L Switch:SW_Push_DPDT SW_Toggle-auto-or-manual?
+U 1 1 5E6F2DFB
+P 2900 4600
+F 0 "SW_Toggle-auto-or-manual?" V 2946 4212 50  0000 R CNN
+F 1 "SW_Push_DPDT" V 2855 4212 50  0000 R CNN
+F 2 "" H 2900 4800 50  0001 C CNN
+F 3 "~" H 2900 4800 50  0001 C CNN
+	1    2900 4600
+	0    -1   -1   0
+$EndComp
+Wire Wire Line
+	2600 4400 2200 4400
+Wire Wire Line
+	2200 4400 2200 3800
+Wire Wire Line
+	3000 4400 3000 4100
+Wire Wire Line
+	3000 4100 2600 4100
+Wire Wire Line
+	2600 4100 2600 3800
+Wire Wire Line
+	3200 4400 4250 4400
+Wire Wire Line
+	4250 4400 4250 4650
+Wire Wire Line
+	2800 4400 2800 4250
+Wire Wire Line
+	2800 4250 4250 4250
+Wire Wire Line
+	2700 4800 2700 4900
+Wire Wire Line
+	2700 4900 2650 4900
+Wire Wire Line
+	2650 4900 2650 5150
+Wire Wire Line
+	3100 4800 3100 4900
+Wire Wire Line
+	3100 4900 3150 4900
+Wire Wire Line
+	3150 4900 3150 5150
+Wire Wire Line
+	2700 3400 2700 2350
+Wire Wire Line
+	2700 2350 3300 2350
+Wire Wire Line
+	4100 2350 4150 2350
+Wire Wire Line
+	4150 2350 4150 2650
+Wire Wire Line
+	4250 2850 2500 2850
+Wire Wire Line
+	2500 2850 2500 3400
+Wire Wire Line
+	3800 2350 3800 3850
+Connection ~ 3800 2350
+Wire Wire Line
+	5000 4350 5000 4750
+Wire Wire Line
+	4100 3850 4100 3100
+Wire Wire Line
+	4100 3100 5200 3100
+Wire Wire Line
+	5200 3100 5200 4350
+Wire Wire Line
+	5200 4350 5000 4350
+Wire Wire Line
+	3800 3850 4100 3850
+Wire Bus Line
+	4050 2750 5800 2750
+Connection ~ 4100 3850
+Wire Wire Line
+	4100 3850 4250 3850
+Connection ~ 5000 4350
 $EndSCHEMATC
